Commit message: tunning and other updates

File: andino/andino_description/urdf/andino.urdf.xacro (robot description, xacro)
@@ -26,9 +26,9 @@
   <xacro:footprint wheel_props="${wheel_props}" />
   <!-- Base link -->
-  <xacro:base link_name="base_link" base_prop="${base_props}" mesh="${base_props['base']['mesh']}" >
+  <xacro:base link_name="base_link" base_prop="${base_props}" mesh="${base_props['base']['mesh']}" radius="${base_props['base']['radius']}" >
     <origin xyz="0 0 0" rpy="0 0 0" />
   </xacro:base>
   <!-- Second story link -->
-  <xacro:base link_name="second_base_link" base_prop="${second_base_props}" mesh="${second_base_props['base']['mesh']}" >
+  <xacro:base link_name="second_base_link" base_prop="${second_base_props}" mesh="${second_base_props['base']['mesh']}" radius="${second_base_props['base']['radius']}" >
     <origin xyz="0 0 0.05" rpy="0 0 0" />
   </xacro:base>

File: andino/andino_description/urdf/include/common_macros.urdf.xacro (robot description, xacro)
@@ -130,11 +130,21 @@
 -->
   <xacro:macro name="base"
-               params="link_name:='base_link' base_prop mesh:='' scale:='' *origin ">
+               params="link_name:='base_link' base_prop mesh:='' scale:='' radius:='' *origin ">
     <link name="${link_name}">
-    <xacro:box_inertia m="${base_prop['base']['mass']}"
-                       x="${base_prop['base']['x_size']}"
-                       y="${base_prop['base']['y_size']}"
-                       z="${base_prop['base']['z_size']}">
-    </xacro:box_inertia>
+    <xacro:if value="${radius != ''}">
+      <xacro:cylinder_inertia m="${base_prop['base']['mass']}"
+                               r="${radius}"
+                               l="${base_prop['base']['z_size']}"
+                               o_xyz="0.0 0.0 0.0"
+                               o_rpy="0.0 0.0 0.0">
+      </xacro:cylinder_inertia>
+    </xacro:if>
+    <xacro:unless value="${radius != ''}">
+      <xacro:box_inertia m="${base_prop['base']['mass']}"
+                         x="${base_prop['base']['x_size']}"
+                         y="${base_prop['base']['y_size']}"
+                         z="${base_prop['base']['z_size']}">
+      </xacro:box_inertia>
+    </xacro:unless>
     <xacro:if value="${mesh != '' }" >
       <visual>
@@ -156,5 +166,10 @@
         <xacro:insert_block name="origin" />
         <geometry>
-          <box size="${base_prop['base']['x_size']} ${base_prop['base']['y_size']} ${base_prop['base']['z_size']}"/>
+          <xacro:if value="${radius != ''}">
+            <cylinder radius="${radius}" length="${base_prop['base']['z_size']}"/>
+          </xacro:if>
+          <xacro:unless value="${radius != ''}">
+            <box size="${base_prop['base']['x_size']} ${base_prop['base']['y_size']} ${base_prop['base']['z_size']}"/>
+          </xacro:unless>
         </geometry>
         <material name="blue" />
@@ -164,5 +179,10 @@
       <origin xyz="0.0 0.0 0.0" rpy="0.0 0.0 0.0"/>
       <geometry>
-        <box size="${base_prop['base']['x_size']} ${base_prop['base']['y_size']} ${base_prop['base']['z_size']}"/>
+        <xacro:if value="${radius != ''}">
+          <cylinder radius="${radius}" length="${base_prop['base']['z_size']}"/>
+        </xacro:if>
+        <xacro:unless value="${radius != ''}">
+          <box size="${base_prop['base']['x_size']} ${base_prop['base']['y_size']} ${base_prop['base']['z_size']}"/>
+        </xacro:unless>
       </geometry>
     </collision>

File: andino_gz/andino_gz/urdf/andino_gz.urdf.xacro (robot description, xacro)
@@ -8,5 +8,5 @@
       <left_joint>left_wheel_joint</left_joint>
       <right_joint>right_wheel_joint</right_joint>
-      <wheel_separation>0.137</wheel_separation>
+      <wheel_separation>0.16</wheel_separation>
       <wheel_radius>0.033</wheel_radius>
       <!--
